File: PCB/Rev 1.0/tNode-8.brd (EAGLE design)
At the start: 157.5 x 97.8 mm, 57 parts, among them IC1 MAX481CSA, J11 C1, J12 D1, J13 C2, J14 D2, J3 A1, J4 B1, J5 A2, J6 B2, U1 9V

Commit message: [WIP] add all UART-DMX outputs
Parts:
- added C10, C11, C12, C13, C14, C15, C16, C41, C42, C43, C44, C45, C46, C47, C48, C49, C50, C51, C52, C53, C54, C55, C56: 0u1, rcl:C0603K
- added C17, C18, C19, C20, C21, C22, C23, C24, C25, C26, C27, C28, C29, C30, C31, C32, C33, C34, C35, C36, C37, C38, C39, C40: 10u, rcl:C0603K
- added C57: 100u, rcl:PANASONIC_D
- added C58: 470u, rcl:PANASONIC_D
- added D10, D11, D12, D13, D14, D15, D16, D9: LM712, diode:SOT23
- added D3, D4, D5, D6, D7, D8: (no value), SparkFun-LED:LED-0603
- added DC3, DC4, DC5, DC6, DC7, DC8: CRE1S0505S3C, dc-dc-converter:4SIL
- added DC9: SHHD003A0A, dc-dc-converter:SHHD003A0A
- added F2, F3, F4, F5, F6, F7, F8: PTC0603, SparkFun-PowerIC:0603
- added IC2, IC3, IC4, IC5, IC6, IC7, IC8: MAX481CSA, maxim:SO08
- added OK2, OK3, OK4, OK5, OK6, OK7, OK8: ACSL-6310, optocoupler:SO-16
- added R15, R16, R17, R18, R19, R20, R21, R22, R23, R24, R25, R26, R27, R28, R29, R30, R31, R32, R33, R34, R35, R36, R37, R38, R39, R40, R41, R42, R43, R44, R45, R46, R47, R48, R49, R50, R51, R52, R53, R54, R55, R56: 470, rcl:R0603
- added R57, R59, R60, R62, R63, R65, R66, R68, R69, R71, R72, R74, R75, R77, R78, R80: 562, rcl:R0603
- added R58, R61, R64, R67, R70, R73, R76, R79: 133, rcl:R0603
- added R81, R82, R83, R84, R85, R86, R87, R88, R89, R90, R91, R92, R93, R94, R95, R96: 10, rcl:R0603
- added R97, R98: 4k7, rcl:R0603
- added U2, U3, U4, U5, U6, U7, U8: 9V, diode:SOD323-NOSILK
- added X1, X6, X7, X8: (no value), con-phoenix-254:3POL254
- added X10: (no value), con-phoenix-254:4POL254
- added X11: (no value), con-phoenix-254:9POL254
- added X9: (no value), con-phoenix-254:2POL254
- C2, C6, C7: value 0u1 -> 10u; device rcl:C0603K -> rcl:E2,5-5-NOSILK
- C3, C4, C5: device rcl:C0603K -> rcl:E2,5-5-NOSILK
- C8: value 100u -> 10u; device rcl:PANASONIC_D -> rcl:E2,5-5-NOSILK
- C9: value 470u -> 0u1; device rcl:PANASONIC_D -> rcl:C0603K
- D2: value LM712 -> (none); device diode:SOT23 -> SparkFun-LED:LED-0603
- DC2: value SHHD003A0A -> CRE1S0505S3C; device dc-dc-converter:SHHD003A0A -> dc-dc-converter:4SIL
- R10, R8: value 562 -> 470
- R11, R12: value 10 -> 470
- R13, R14: value 4k7 -> 470
- R9: value 133 -> 470
- X3: device con-phoenix-254:2POL254 -> con-phoenix-254:3POL254
- X4: device con-phoenix-254:4POL254 -> con-phoenix-254:3POL254
- X5: device con-phoenix-254:9POL254 -> con-phoenix-254:3POL254
- moved C8 160.3 mm to (151.1, 26.7), turned to 180 degrees
- moved R8 126.2 mm to (141.0, 27.3), turned to 0 degrees
- moved C7 122.2 mm to (132.1, 26.7), turned to 180 degrees
- moved R7 109.5 mm to (121.9, 27.3), turned to 0 degrees
- moved C6 103.7 mm to (113.0, 26.7), turned to 180 degrees
- moved X3 100.5 mm to (51.4, 2.54), turned to 180 degrees
- moved R6 96.4 mm to (102.9, 27.3), turned to 0 degrees
- moved X4 96.3 mm to (70.5, 2.54), turned to 180 degrees
- moved R5 77.7 mm to (83.8, 27.3), turned to 0 degrees
- moved C5 77.3 mm to (94.0, 26.7), turned to 180 degrees
- moved R13 69.9 mm to (29.2, 23.5), turned to 0 degrees
- moved R14 68.7 mm to (26.7, 24.8), turned to 0 degrees
- moved C4 58.5 mm to (74.9, 26.7), turned to 180 degrees
- moved DC2 58.4 mm to (36.2, 18.4)
- moved R4 54.0 mm to (64.8, 27.3)
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Connections:
- removed net +5V-1: C4.1, C5.1, C6.1, C7.1, DC1.4, IC1.8, OK1.12, R10.2, R5.1, R6.1, R7.1
- removed net GND-ISO: C4.2, C5.2, C6.2, C7.2, D2.3, DC1.3, IC1.5, OK1.9, R8.1, X2.1
- new net +5V-ISO1: C25.1, C33.1, C41.1, C49.1, DC1.4, IC1.8, OK1.12, R33.1, R34.1, R35.1, R59.2
- new net +5V-ISO2: C26.1, C34.1, C42.1, C50.1, DC2.4, IC2.8, OK2.12, R36.1, R37.1, R38.1, R62.2
- new net +5V-ISO3: C27.1, C35.1, C43.1, C51.1, DC3.4, IC3.8, OK3.12, R39.1, R40.1, R41.1, R65.2
- new net +5V-ISO4: C28.1, C36.1, C44.1, C52.1, DC4.4, IC4.8, OK4.12, R42.1, R43.1, R44.1, R68.2
- new net +5V-ISO5: C29.1, C37.1, C45.1, C53.1, DC5.4, IC5.8, OK5.12, R45.1, R46.1, R47.1, R71.2
- new net +5V-ISO6: C30.1, C38.1, C46.1, C54.1, DC6.4, IC6.8, OK6.12, R48.1, R49.1, R50.1, R74.2
- new net +5V-ISO7: C31.1, C39.1, C47.1, C55.1, DC7.4, IC7.8, OK7.12, R51.1, R52.1, R53.1, R77.2
- new net +5V-ISO8: C32.1, C40.1, C48.1, C56.1, DC8.4, IC8.8, OK8.12, R54.1, R55.1, R56.1, R80.2
- new net GND-ISO1: C25.2, C33.2, C41.2, C49.2, D9.3, DC1.3, IC1.5, OK1.9, R57.1, X1.1
- new net GND-ISO2: C26.2, C34.2, C42.2, C50.2, D10.3, DC2.3, IC2.5, OK2.9, R60.1, X2.1
- new net GND-ISO3: C27.2, C35.2, C43.2, C51.2, D11.3, DC3.3, IC3.5, OK3.9, R63.1, X3.1
- new net GND-ISO4: C28.2, C36.2, C44.2, C52.2, D12.3, DC4.3, IC4.5, OK4.9, R66.1, X4.1
- new net GND-ISO5: C29.2, C37.2, C45.2, C53.2, D13.3, DC5.3, IC5.5, OK5.9, R69.1, X5.1
- new net GND-ISO6: C30.2, C38.2, C46.2, C54.2, D14.3, DC6.3, IC6.5, OK6.9, R72.1, X6.1
- new net GND-ISO7: C31.2, C39.2, C47.2, C55.2, D15.3, DC7.3, IC7.5, OK7.9, R75.1, X7.1
- new net GND-ISO8: C32.2, C40.2, C48.2, C56.2, D16.3, DC8.3, IC8.5, OK8.9, R78.1, X8.1
- new net N$1: IC2.7, R60.2, R61.1, R83.1
- new net N$11: D2.C, R2.1
- new net N$12: D10.1, R83.2, X2.2
- new net N$13: D10.2, R84.2, X2.3
- new net N$14: IC3.7, R63.2, R64.1, R85.1
- new net N$15: IC3.6, R64.2, R65.1, R86.1
- new net N$16: IC3.1, OK3.13
- new net N$17: IC3.2, IC3.3, OK3.11, R40.2
- new net N$20: OK3.5, R16.1
- new net N$22: OK3.7, R17.1
- new net N$24: OK3.14, R39.2
- new net N$26: D3.C, R3.1
- new net N$29: D11.1, R85.2, X3.2
- new net N$30: D11.2, R86.2, X3.3
- new net N$31: IC4.7, R66.2, R67.1, R87.1
- new net N$33: IC4.6, R67.2, R68.1, R88.1
- new net N$35: IC4.1, OK4.13
- new net N$36: IC4.2, IC4.3, OK4.11, R43.2
- new net N$37: OK4.5, R19.1
- new net N$38: OK4.7, R20.1
- new net N$39: OK4.14, R42.2
- new net N$4: IC2.6, R61.2, R62.1, R84.1
- new net N$40: D4.C, R4.1
- new net N$41: D12.1, R87.2, X4.2
- new net N$42: D12.2, R88.2, X4.3
- new net N$43: IC5.7, R69.2, R70.1, R89.1
- new net N$44: IC5.6, R70.2, R71.1, R90.1
- new net N$45: IC5.1, OK5.13
- new net N$46: IC5.2, IC5.3, OK5.11, R46.2
- new net N$47: OK5.5, R22.1
- new net N$48: OK5.7, R23.1
- new net N$49: OK5.14, R45.2
- new net N$5: IC2.1, OK2.13
- new net N$50: D5.C, R5.1
- new net N$51: D13.1, R89.2, X5.2
- new net N$52: D13.2, R90.2, X5.3
- new net N$53: IC6.7, R72.2, R73.1, R91.1
- new net N$54: IC6.6, R73.2, R74.1, R92.1
- new net N$55: IC6.1, OK6.13
- new net N$56: IC6.2, IC6.3, OK6.11, R49.2
- new net N$57: OK6.5, R25.1
- new net N$58: OK6.7, R26.1
- new net N$59: OK6.14, R48.2
- new net N$6: IC2.2, IC2.3, OK2.11, R37.2
- new net N$60: D6.C, R6.1
- new net N$61: D14.1, R91.2, X6.2
- new net N$62: D14.2, R92.2, X6.3
- new net N$63: IC7.7, R75.2, R76.1, R93.1
- new net N$64: IC7.6, R76.2, R77.1, R94.1
- new net N$65: IC7.1, OK7.13
- new net N$66: IC7.2, IC7.3, OK7.11, R52.2
- new net N$67: OK7.5, R28.1
- new net N$68: OK7.7, R29.1
- new net N$69: OK7.14, R51.2
- new net N$7: OK2.5, R13.1
- new net N$70: D7.C, R7.1
- new net N$71: D15.1, R93.2, X7.2
- new net N$72: D15.2, R94.2, X7.3
- new net N$73: IC8.7, R78.2, R79.1, R95.1
- new net N$74: IC8.6, R79.2, R80.1, R96.1
- new net N$75: IC8.1, OK8.13
- new net N$76: IC8.2, IC8.3, OK8.11, R55.2
- new net N$77: OK8.5, R31.1
- new net N$78: OK8.7, R32.1
- new net N$79: OK8.14, R54.2
- new net N$8: OK2.7, R14.1
- new net N$80: D8.C, R8.1
- new net N$81: D16.1, R95.2, X8.2
- new net N$82: D16.2, R96.2, X8.3
- new net N$9: OK2.14, R36.2
- new net OPTO-OUT2: IC2.4, OK2.10, R38.2
- new net OPTO-OUT3: IC3.4, OK3.10, R41.2
- new net OPTO-OUT4: IC4.4, OK4.10, R44.2
- new net OPTO-OUT5: IC5.4, OK5.10, R47.2
- new net OPTO-OUT6: IC6.4, OK6.10, R50.2
- new net OPTO-OUT7: IC7.4, OK7.10, R53.2
- new net OPTO-OUT8: IC8.4, OK8.10, R56.2
- new net VIN-2: C10.1, C18.1, C2.+, D2.A, DC2.2, F2.2, OK2.4, R12.1, R13.2, R14.2, U2.C
- new net VIN-3: C11.1, C19.1, C3.+, D3.A, DC3.2, F3.2, OK3.4, R15.1, R16.2, R17.2, U3.C
- new net VIN-4: C12.1, C20.1, C4.+, D4.A, DC4.2, F4.2, OK4.4, R18.1, R19.2, R20.2, U4.C
- new net VIN-5: C13.1, C21.1, C5.+, D5.A, DC5.2, F5.2, OK5.4, R21.1, R22.2, R23.2, U5.C
- new net VIN-6: C14.1, C22.1, C6.+, D6.A, DC6.2, F6.2, OK6.4, R24.1, R25.2, R26.2, U6.C
- new net VIN-7: C15.1, C23.1, C7.+, D7.A, DC7.2, F7.2, OK7.4, R27.1, R28.2, R29.2, U7.C
- new net VIN-8: C16.1, C24.1, C8.+, D8.A, DC8.2, F8.2, OK8.4, R30.1, R31.2, R32.2, U8.C
- net 5V: now also C58.+, DC9.4, F2.1, F3.1, F4.1, F5.1, F6.1, F7.1, F8.1, R97.2, R98.2, X10.4; no longer C9.+, DC2.4, R13.2, R14.2, X4.4
- net GND: now also C10.2, C11.2, C12.2, C13.2, C14.2, C15.2, C16.2, C17.2, C18.2, C19.2, C2.-, C20.2, C21.2, C22.2, C23.2, C24.2, C3.-, C4.-, C5.-, C58.-, C6.-, C7.-, C8.-, C9.2, DC2.1, DC3.1, DC4.1, DC5.1, DC6.1, DC7.1, DC8.1, DC9.6, OK2.1, OK3.1, OK4.1, OK5.1, OK6.1, OK7.1, OK8.1, R2.2, R3.2, R4.2, R5.2, R6.2, R7.2, R8.2, U2.A, U3.A, U4.A, U5.A, U6.A, U7.A, U8.A, X10.1, X11.1; no longer C2.2, C3.2, C9.-, DC2.6, X4.1, X5.1
- net I2C0-SCL: now also R98.1, X10.2; no longer R14.1, X4.2
- net I2C0-SDA: now also R97.1, X10.3; no longer R13.1, X4.3
- net N$18: now also R34.2; no longer R5.2
- net N$19: now also R10.1; no longer R2.1
- net N$2: now also R57.2, R58.1, R81.1; no longer R11.1, R8.2, R9.1
- net N$21: now also R11.1; no longer R3.1
- net N$23: now also R33.2; no longer R7.2
- net N$27: now also D9.1, R81.2, X1.2; no longer D2.1, R11.2, X2.2
- net N$28: now also D9.2, R82.2, X1.3; no longer D2.2, R12.2, X2.3
- net N$3: now also R58.2, R59.1, R82.1; no longer R10.1, R12.1, R9.2
- net N$32: now also C57.-, DC9.1, X9.2; no longer C8.-, DC2.1, X3.2
- net N$34: now also C57.+, DC9.3, X9.1; no longer C8.+, DC2.3, X3.1
- net OPTO-OUT1: now also R35.2; no longer R6.2
- net U0RX: now also OK2.3, OK3.3, OK4.3, OK5.3, OK6.3, OK7.3, OK8.3, R12.2, R15.2, R18.2, R21.2, R24.2, R27.2, R30.2, R9.2; no longer R4.2
- net U0SEL: now also OK2.6, OK3.6, OK4.6, OK5.6, OK6.6, OK7.6, OK8.6
- net U0TX: now also OK2.8, OK3.8, OK4.8, OK5.8, OK6.8, OK7.8, OK8.8, X11.9; no longer X5.9
- net U1TX: now also X11.8; no longer X5.8
- net U2TX: now also X11.7; no longer X5.7
- net U3TX: now also X11.6; no longer X5.6
- net U4TX: now also X11.5; no longer X5.5
- net U5TX: now also X11.4; no longer X5.4
- net U6TX: now also X11.3; no longer X5.3
- net U7TX: now also X11.2; no longer X5.2
- net VIN-1: now also C17.1, C9.1, R10.2, R11.2, R9.1; no longer C2.1, C3.1, R2.2, R3.2, R4.1
Routing:
- net U0RX: track 9.89 -> 79.1 mm
- net U0SEL: track 9.25 -> 74.0 mm
- net U0TX: track 8.99 -> 71.9 mm
- net VIN-8: track 0.00 -> 33.9 mm, vias 0 -> 2
- net VIN-6: track 0.00 -> 33.9 mm, vias 0 -> 2
- net VIN-5: track 0.00 -> 33.9 mm, vias 0 -> 2
- net VIN-4: track 0.00 -> 33.9 mm, vias 0 -> 2
- net VIN-3: track 0.00 -> 33.9 mm, vias 0 -> 2
- net VIN-2: track 0.00 -> 33.9 mm, vias 0 -> 2
- net VIN-7: track 0.00 -> 33.9 mm, vias 0 -> 2
- net +5V-ISO8: track 0.00 -> 31.7 mm, vias 0 -> 1
- net +5V-ISO7: track 0.00 -> 31.7 mm, vias 0 -> 1
- net +5V-ISO5: track 0.00 -> 31.7 mm, vias 0 -> 1
- net +5V-ISO3: track 0.00 -> 31.7 mm, vias 0 -> 1
- net +5V-ISO4: track 0.00 -> 31.7 mm, vias 0 -> 1
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- added copper zone on layer 1, net GND-ISO1
- added copper zone on layer 16, net GND-ISO1
- added copper zone on layer 1, net GND-ISO2
- added copper zone on layer 16, net GND-ISO2
- added copper zone on layer 1, net GND-ISO3
- added copper zone on layer 16, net GND-ISO3
- added copper zone on layer 1, net GND-ISO4
- added copper zone on layer 16, net GND-ISO4
- added copper zone on layer 1, net GND-ISO5
- added copper zone on layer 16, net GND-ISO5
- added copper zone on layer 1, net GND-ISO6
- added copper zone on layer 16, net GND-ISO6
- added copper zone on layer 1, net GND-ISO7
- added copper zone on layer 16, net GND-ISO7
- added copper zone on layer 1, net GND-ISO8
- added copper zone on layer 16, net GND-ISO8
- removed copper zone on layer 1, net GND-ISO
- removed copper zone on layer 16, net GND-ISO
Other:
- board size 157.5 x 97.8 mm -> 158.8 x 97.8 mm
