File: PCB/Rev 1.0/tNode-8.sch (EAGLE design)
At the start: 57 parts, among them IC1 MAX481CSA, J11 C1, J12 D1, J13 C2, J14 D2, J3 A1, J4 B1, J5 A2, J6 B2, U1 9V

Commit message: [WIP] add all UART-DMX outputs
Parts:
- added C10, C11, C12, C13, C14, C15, C16, C41, C42, C43, C44, C45, C46, C47, C48, C49, C50, C51, C52, C53, C54, C55, C56: 0u1, rcl:C-USC0603K
- added C17, C18, C19, C20, C21, C22, C23, C24, C25, C26, C27, C28, C29, C30, C31, C32, C33, C34, C35, C36, C37, C38, C39, C40: 10u, rcl:C-USC0603K
- added C57: 100u, rcl:CPOL-USD
- added C58: 470u, rcl:CPOL-USD
- added D10, D11, D12, D13, D14, D15, D16, D9: LM712, diode:CDSOT23-SM712SOT23-STANDARD
- added D3, D4, D5, D6, D7, D8: (no value), SparkFun-LED:LED0603
- added DC3, DC4, DC5, DC6, DC7, DC8: CRE1S0505S3C, dc-dc-converter:VA-0505S
- added DC9: SHHD003A0A, dc-dc-converter:SHHD003A0A
- added F2, F3, F4, F5, F6, F7, F8: PTC0603, SparkFun-PowerIC:PTC0603
- added IC2, IC3, IC4, IC5, IC6, IC7, IC8: MAX481CSA, maxim:MAX481CSA
- added OK2, OK3, OK4, OK5, OK6, OK7, OK8: ACSL-6310, optocoupler:ACSL-60
- added R15, R16, R17, R18, R19, R20, R21, R22, R23, R24, R25, R26, R27, R28, R29, R30, R31, R32, R33, R34, R35, R36, R37, R38, R39, R40, R41, R42, R43, R44, R45, R46, R47, R48, R49, R50, R51, R52, R53, R54, R55, R56: 470, rcl:R-US_R0603
- added R57, R59, R60, R62, R63, R65, R66, R68, R69, R71, R72, R74, R75, R77, R78, R80: 562, rcl:R-US_R0603
- added R58, R61, R64, R67, R70, R73, R76, R79: 133, rcl:R-US_R0603
- added R81, R82, R83, R84, R85, R86, R87, R88, R89, R90, R91, R92, R93, R94, R95, R96: 10, rcl:R-US_R0603
- added R97, R98: 4k7, rcl:R-US_R0603
- added U2, U3, U4, U5, U6, U7, U8: 9V, diode:TVS-DIODESOD323-NOSILK
- added X1, X6, X7, X8: (no value), con-phoenix-254:MPT3
- added X10: (no value), con-phoenix-254:MPT4
- added X11: (no value), con-phoenix-254:MPT9
- added X9: (no value), con-phoenix-254:MPT2
- C2, C6, C7: value 0u1 -> 10u; device rcl:C-USC0603K -> rcl:CPOL-USE2.5-5-NOSILK
- C3, C4, C5: device rcl:C-USC0603K -> rcl:CPOL-USE2.5-5-NOSILK
- C8: value 100u -> 10u; device rcl:CPOL-USD -> rcl:CPOL-USE2.5-5-NOSILK
- C9: value 470u -> 0u1; device rcl:CPOL-USD -> rcl:C-USC0603K
- D2: value LM712 -> (none); device diode:CDSOT23-SM712SOT23-STANDARD -> SparkFun-LED:LED0603
- DC2: value SHHD003A0A -> CRE1S0505S3C; device dc-dc-converter:SHHD003A0A -> dc-dc-converter:VA-0505S
- R10, R8: value 562 -> 470
- R11, R12: value 10 -> 470
- R13, R14: value 4k7 -> 470
- R9: value 133 -> 470
- X3: device con-phoenix-254:MPT2 -> con-phoenix-254:MPT3
- X4: device con-phoenix-254:MPT4 -> con-phoenix-254:MPT3
- X5: device con-phoenix-254:MPT9 -> con-phoenix-254:MPT3
Connections:
- removed net +5V-1: C4.1, C5.1, C6.1, C7.1, DC1.+VOUT, IC1P.VCC, OK1.VDD2, R10.2, R5.1, R6.1, R7.1
- removed net GND-ISO: C4.2, C5.2, C6.2, C7.2, D2.3, DC1.-VOUT, IC1P.GND, OK1.GND2, R8.1, X2-1.1
- new net +5V-ISO1: C25.1, C33.1, C41.1, C49.1, DC1.+VOUT, IC1P.VCC, OK1.VDD2, R33.1, R34.1, R35.1, R59.2
- new net +5V-ISO2: C26.1, C34.1, C42.1, C50.1, DC2.+VOUT, IC2P.VCC, OK2.VDD2, R36.1, R37.1, R38.1, R62.2
- new net +5V-ISO3: C27.1, C35.1, C43.1, C51.1, DC3.+VOUT, IC3P.VCC, OK3.VDD2, R39.1, R40.1, R41.1, R65.2
- new net +5V-ISO4: C28.1, C36.1, C44.1, C52.1, DC4.+VOUT, IC4P.VCC, OK4.VDD2, R42.1, R43.1, R44.1, R68.2
- new net +5V-ISO5: C29.1, C37.1, C45.1, C53.1, DC5.+VOUT, IC5P.VCC, OK5.VDD2, R45.1, R46.1, R47.1, R71.2
- new net +5V-ISO6: C30.1, C38.1, C46.1, C54.1, DC6.+VOUT, IC6P.VCC, OK6.VDD2, R48.1, R49.1, R50.1, R74.2
- new net +5V-ISO7: C31.1, C39.1, C47.1, C55.1, DC7.+VOUT, IC7P.VCC, OK7.VDD2, R51.1, R52.1, R53.1, R77.2
- new net +5V-ISO8: C32.1, C40.1, C48.1, C56.1, DC8.+VOUT, IC8P.VCC, OK8.VDD2, R54.1, R55.1, R56.1, R80.2
- new net GND-ISO1: C25.2, C33.2, C41.2, C49.2, D9.3, DC1.-VOUT, IC1P.GND, OK1.GND2, R57.1, X1-1.1
- new net GND-ISO2: C26.2, C34.2, C42.2, C50.2, D10.3, DC2.-VOUT, IC2P.GND, OK2.GND2, R60.1, X2-1.1
- new net GND-ISO3: C27.2, C35.2, C43.2, C51.2, D11.3, DC3.-VOUT, IC3P.GND, OK3.GND2, R63.1, X3-1.1
- new net GND-ISO4: C28.2, C36.2, C44.2, C52.2, D12.3, DC4.-VOUT, IC4P.GND, OK4.GND2, R66.1, X4-1.1
- new net GND-ISO5: C29.2, C37.2, C45.2, C53.2, D13.3, DC5.-VOUT, IC5P.GND, OK5.GND2, R69.1, X5-1.1
- new net GND-ISO6: C30.2, C38.2, C46.2, C54.2, D14.3, DC6.-VOUT, IC6P.GND, OK6.GND2, R72.1, X6-1.1
- new net GND-ISO7: C31.2, C39.2, C47.2, C55.2, D15.3, DC7.-VOUT, IC7P.GND, OK7.GND2, R75.1, X7-1.1
- new net GND-ISO8: C32.2, C40.2, C48.2, C56.2, D16.3, DC8.-VOUT, IC8P.GND, OK8.GND2, R78.1, X8-1.1
- new net N$1: IC2G$1.B, R60.2, R61.1, R83.1
- new net N$11: D2.C, R2.1
- new net N$12: D10.1, R83.2, X2-2.1
- new net N$13: D10.2, R84.2, X2-3.1
- new net N$14: IC3G$1.B, R63.2, R64.1, R85.1
- new net N$15: IC3G$1.A, R64.2, R65.1, R86.1
- new net N$16: IC3G$1.RO, OK3.C3
- new net N$17: IC3G$1.DE, IC3G$1.RE/, OK3.VO1, R40.2
- new net N$20: OK3.A1, R16.1
- new net N$22: OK3.A2, R17.1
- new net N$24: OK3.A3, R39.2
- new net N$26: D3.C, R3.1
- new net N$29: D11.1, R85.2, X3-2.1
- new net N$30: D11.2, R86.2, X3-3.1
- new net N$31: IC4G$1.B, R66.2, R67.1, R87.1
- new net N$33: IC4G$1.A, R67.2, R68.1, R88.1
- new net N$35: IC4G$1.RO, OK4.C3
- new net N$36: IC4G$1.DE, IC4G$1.RE/, OK4.VO1, R43.2
- new net N$37: OK4.A1, R19.1
- new net N$38: OK4.A2, R20.1
- new net N$39: OK4.A3, R42.2
- new net N$4: IC2G$1.A, R61.2, R62.1, R84.1
- new net N$40: D4.C, R4.1
- new net N$41: D12.1, R87.2, X4-2.1
- new net N$42: D12.2, R88.2, X4-3.1
- new net N$43: IC5G$1.B, R69.2, R70.1, R89.1
- new net N$44: IC5G$1.A, R70.2, R71.1, R90.1
- new net N$45: IC5G$1.RO, OK5.C3
- new net N$46: IC5G$1.DE, IC5G$1.RE/, OK5.VO1, R46.2
- new net N$47: OK5.A1, R22.1
- new net N$48: OK5.A2, R23.1
- new net N$49: OK5.A3, R45.2
- new net N$5: IC2G$1.RO, OK2.C3
- new net N$50: D5.C, R5.1
- new net N$51: D13.1, R89.2, X5-2.1
- new net N$52: D13.2, R90.2, X5-3.1
- new net N$53: IC6G$1.B, R72.2, R73.1, R91.1
- new net N$54: IC6G$1.A, R73.2, R74.1, R92.1
- new net N$55: IC6G$1.RO, OK6.C3
- new net N$56: IC6G$1.DE, IC6G$1.RE/, OK6.VO1, R49.2
- new net N$57: OK6.A1, R25.1
- new net N$58: OK6.A2, R26.1
- new net N$59: OK6.A3, R48.2
- new net N$6: IC2G$1.DE, IC2G$1.RE/, OK2.VO1, R37.2
- new net N$60: D6.C, R6.1
- new net N$61: D14.1, R91.2, X6-2.1
- new net N$62: D14.2, R92.2, X6-3.1
- new net N$63: IC7G$1.B, R75.2, R76.1, R93.1
- new net N$64: IC7G$1.A, R76.2, R77.1, R94.1
- new net N$65: IC7G$1.RO, OK7.C3
- new net N$66: IC7G$1.DE, IC7G$1.RE/, OK7.VO1, R52.2
- new net N$67: OK7.A1, R28.1
- new net N$68: OK7.A2, R29.1
- new net N$69: OK7.A3, R51.2
- new net N$7: OK2.A1, R13.1
- new net N$70: D7.C, R7.1
- new net N$71: D15.1, R93.2, X7-2.1
- new net N$72: D15.2, R94.2, X7-3.1
- new net N$73: IC8G$1.B, R78.2, R79.1, R95.1
- new net N$74: IC8G$1.A, R79.2, R80.1, R96.1
- new net N$75: IC8G$1.RO, OK8.C3
- new net N$76: IC8G$1.DE, IC8G$1.RE/, OK8.VO1, R55.2
- new net N$77: OK8.A1, R31.1
- new net N$78: OK8.A2, R32.1
- new net N$79: OK8.A3, R54.2
- new net N$8: OK2.A2, R14.1
- new net N$80: D8.C, R8.1
- new net N$81: D16.1, R95.2, X8-2.1
- new net N$82: D16.2, R96.2, X8-3.1
- new net N$9: OK2.A3, R36.2
- new net OPTO-OUT2: IC2G$1.DI, OK2.VO2, R38.2
- new net OPTO-OUT3: IC3G$1.DI, OK3.VO2, R41.2
- new net OPTO-OUT4: IC4G$1.DI, OK4.VO2, R44.2
- new net OPTO-OUT5: IC5G$1.DI, OK5.VO2, R47.2
- new net OPTO-OUT6: IC6G$1.DI, OK6.VO2, R50.2
- new net OPTO-OUT7: IC7G$1.DI, OK7.VO2, R53.2
- new net OPTO-OUT8: IC8G$1.DI, OK8.VO2, R56.2
- new net VIN-2: C10.1, C18.1, C2.+, D2.A, DC2.+VIN, F2.2, OK2.VDD1, R12.1, R13.2, R14.2, U2.C
- new net VIN-3: C11.1, C19.1, C3.+, D3.A, DC3.+VIN, F3.2, OK3.VDD1, R15.1, R16.2, R17.2, U3.C
- new net VIN-4: C12.1, C20.1, C4.+, D4.A, DC4.+VIN, F4.2, OK4.VDD1, R18.1, R19.2, R20.2, U4.C
- new net VIN-5: C13.1, C21.1, C5.+, D5.A, DC5.+VIN, F5.2, OK5.VDD1, R21.1, R22.2, R23.2, U5.C
- new net VIN-6: C14.1, C22.1, C6.+, D6.A, DC6.+VIN, F6.2, OK6.VDD1, R24.1, R25.2, R26.2, U6.C
- new net VIN-7: C15.1, C23.1, C7.+, D7.A, DC7.+VIN, F7.2, OK7.VDD1, R27.1, R28.2, R29.2, U7.C
- new net VIN-8: C16.1, C24.1, C8.+, D8.A, DC8.+VIN, F8.2, OK8.VDD1, R30.1, R31.2, R32.2, U8.C
- net 5V: now also C58.+, DC9.VOUT+, F2.1, F3.1, F4.1, F5.1, F6.1, F7.1, F8.1, R97.2, R98.2, X10-4.1; no longer C9.+, DC2.VOUT+, R13.2, R14.2, X4-4.1
- net GND: now also C10.2, C11.2, C12.2, C13.2, C14.2, C15.2, C16.2, C17.2, C18.2, C19.2, C2.-, C20.2, C21.2, C22.2, C23.2, C24.2, C3.-, C4.-, C5.-, C58.-, C6.-, C7.-, C8.-, C9.2, DC2.-VIN, DC3.-VIN, DC4.-VIN, DC5.-VIN, DC6.-VIN, DC7.-VIN, DC8.-VIN, DC9.VOUT-, OK2.GND1, OK3.GND1, OK4.GND1, OK5.GND1, OK6.GND1, OK7.GND1, OK8.GND1, R2.2, R3.2, R4.2, R5.2, R6.2, R7.2, R8.2, U2.A, U3.A, U4.A, U5.A, U6.A, U7.A, U8.A, X10-1.1, X11-1.1; no longer C2.2, C3.2, C9.-, DC2.VOUT-, X4-1.1, X5-1.1
- net I2C0-SCL: now also R98.1, X10-2.1; no longer R14.1, X4-2.1
- net I2C0-SDA: now also R97.1, X10-3.1; no longer R13.1, X4-3.1
- net N$18: now also R34.2; no longer R5.2
- net N$19: now also R10.1; no longer R2.1
- net N$2: now also R57.2, R58.1, R81.1; no longer R11.1, R8.2, R9.1
- net N$21: now also R11.1; no longer R3.1
- net N$23: now also R33.2; no longer R7.2
- net N$27: now also D9.1, R81.2, X1-2.1; no longer D2.1, R11.2, X2-2.1
- net N$28: now also D9.2, R82.2, X1-3.1; no longer D2.2, R12.2, X2-3.1
- net N$3: now also R58.2, R59.1, R82.1; no longer R10.1, R12.1, R9.2
- net N$32: now also C57.-, DC9.VIN-, X9-2.1; no longer C8.-, DC2.VIN-, X3-2.1
- net N$34: now also C57.+, DC9.VIN+, X9-1.1; no longer C8.+, DC2.VIN+, X3-1.1
- net OPTO-OUT1: now also R35.2; no longer R6.2
- net U0RX: now also OK2.V03, OK3.V03, OK4.V03, OK5.V03, OK6.V03, OK7.V03, OK8.V03, R12.2, R15.2, R18.2, R21.2, R24.2, R27.2, R30.2, R9.2; no longer R4.2
- net U0SEL: now also OK2.C1, OK3.C1, OK4.C1, OK5.C1, OK6.C1, OK7.C1, OK8.C1
- net U0TX: now also OK2.C2, OK3.C2, OK4.C2, OK5.C2, OK6.C2, OK7.C2, OK8.C2, X11-9.1; no longer X5-9.1
- net U1TX: now also X11-8.1; no longer X5-8.1
- net U2TX: now also X11-7.1; no longer X5-7.1
- net U3TX: now also X11-6.1; no longer X5-6.1
- net U4TX: now also X11-5.1; no longer X5-5.1
- net U5TX: now also X11-4.1; no longer X5-4.1
- net U6TX: now also X11-3.1; no longer X5-3.1
- net U7TX: now also X11-2.1; no longer X5-2.1
- net VIN-1: now also C17.1, C9.1, R10.2, R11.2, R9.1; no longer C2.1, C3.1, R2.2, R3.2, R4.1
